Commit message: klampt : add liquide urdf, add all type of plateau elect

File: klampt/urdf/sysmap_liquide.urdf (robot description, URDF)
Before this commit: robot sysmap, 21 links, 20 joints
Links:
- removed link stockage_boite
- removed link stockage_boite2
- removed link stockage_boite3
- removed link stockage_couvercle
- removed link stockage_couvercle2
- removed link stockage_couvercle3
- added link stockage_liquide; collision mesh filename=package://klampt/meshes/3_ZoneStockage_liquide_convexHull.s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; visual mesh filename=package://klampt/meshes/3_ZoneStockage_liquide_optimized.stl
- added link stockage_liquide2; collision mesh filename=package://klampt/meshes/3_ZoneStockage_liquide_convexHull.s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; visual mesh filename=package://klampt/meshes/3_ZoneStockage_liquide_optimized.stl
- added link stockage_liquide3; collision mesh filename=package://klampt/meshes/3_ZoneStockage_liquide_convexHull.s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; visual mesh filename=package://klampt/meshes/3_ZoneStockage_liquide_optimized.stl
Joints:
- removed joint platine_stockageBoite
- removed joint platine_stockageBoite2
- removed joint platine_stockageBoite3
- removed joint stockageBoite_couvercle
- removed joint stockageBoite_couvercle2
- removed joint stockageBoite_couvercle3
- added joint platine_stockageLiquide: type fixed, parent platine, child stockage_liquide, origin xyz=-0.2789 -0.06397 0.0 rpy=0.0 0.0 0.0
- added joint platine_stockageLiquide2: type fixed, parent platine, child stockage_liquide2, origin xyz=-0.2789 0.05803 0.0 rpy=0.0 0.0 0.0
- added joint platine_stockageLiquide3: type fixed, parent platine, child stockage_liquide3, origin xyz=-0.2789 0.18003 0.0 rpy=0.0 0.0 0.0
