Commit message: klampt : pince fini

File: klampt/urdf/sysmap2_ros.urdf (robot description, URDF)
Before this commit: robot sysmap, 13 links, 12 joints
Links:
- removed link pince
- removed link poigner
- added link doigt1; collision mesh filename=package://klampt/meshes/7_7_scara_pince_doigt_convexHull.stl; visual mesh filename=package://klampt/meshes/7_7_scara_pince_doigt_optimized.stl
- added link doigt2; collision mesh filename=package://klampt/meshes/7_7_scara_pince_doigt_convexHull.stl; visual mesh filename=package://klampt/meshes/7_7_scara_pince_doigt_optimized.stl
- added link doigt3; collision mesh filename=package://klampt/meshes/7_7_scara_pince_doigt_convexHull.stl; visual mesh filename=package://klampt/meshes/7_7_scara_pince_doigt_optimized.stl
- added link pince_base; collision mesh filename=package://klampt/meshes/7_7_scara_pince_base_convexHull.stl; visual mesh filename=package://klampt/meshes/7_7_scara_pince_base_optimized.stl
- added link poignet; collision mesh filename=package://klampt/meshes/7_5_scara_poignet_convexHull.stl; visual mesh filename=package://klampt/meshes/7_5_scara_poignet_optimized.stl
Joints:
- removed joint externe_poigner
- removed joint poigner_verin
- added joint externe_poignet: type revolute, parent externe, child poignet, origin xyz=0.29117 0.13275 0.030 rpy=0.0 0.0 0.0, axis 0.0 0.0 1.0, limit lower=-6 upper=6 effort=0.0 velocity=0.0
- added joint pince_doigt1: type revolute, parent pince_base, child doigt1, origin xyz=0.02405 0.07176 0.05466 rpy=0.0 2.094 0.0, axis 0.0 0.0 1.0, limit lower=0 upper=0.8346 effort=0.0 velocity=0.0
- added joint pince_doigt2: type revolute, parent pince_base, child doigt2, origin xyz=-0.05936 0.07176 -0.0065 rpy=0.0 0.0 0.0, axis 0.0 0.0 1.0, limit lower=0 upper=0.8346 effort=0.0 velocity=0.0, mimic joint=pince_doigt1 multiplier=1 offset=0
- added joint pince_doigt3: type revolute, parent pince_base, child doigt3, origin xyz=0.03531 0.07176 -0.04816 rpy=0.0 -2.094 0.0, axis 0.0 0.0 1.0, limit lower=0 upper=0.8346 effort=0.0 velocity=0.0, mimic joint=pince_doigt1 multiplier=1 offset=0
- added joint poignet_verin: type prismatic, parent poignet, child verin, origin xyz=0.0 0.0 -0.083 rpy=0.0 0.0 0.0, axis 0.0 0.0 1.0, limit lower=-0.15 upper=0.0 effort=0.0 velocity=0.0
- joint verin_pince: child pince -> pince_base

Commit message: moveit : pince fini

File: klampt/urdf/sysmap2_ros.urdf (robot description, URDF)
Before this commit: robot sysmap, 16 links, 15 joints
Links:
- link interne: geometry collision mesh filename=package://klampt/meshes/7_3_scara_interne_V2_convexHull.stl; visual mesh filename=package://klampt/meshes/7_3_scara_interne_optimized.stl
Joints:
- joint colonne_interne: limit lower=-0.309 upper=0 effort=0.0 velocity=0.0 -> lower=-0.2995 upper=0 effort=0.0 velocity=0.0

File: moveit/config/gazebo_sysmap.urdf (robot description, URDF)
Before this commit: robot sysmap, 13 links, 12 joints
Links:
- removed link pince
- removed link poigner
- added link doigt1, mass 0.1; collision mesh filename=package://klampt/meshes/7_7_scara_pince_doigt_convexHull.stl; visual mesh filename=package://klampt/meshes/7_7_scara_pince_doigt_optimized.stl
- added link doigt2, mass 0.1; collision mesh filename=package://klampt/meshes/7_7_scara_pince_doigt_convexHull.stl; visual mesh filename=package://klampt/meshes/7_7_scara_pince_doigt_optimized.stl
- added link doigt3, mass 0.1; collision mesh filename=package://klampt/meshes/7_7_scara_pince_doigt_convexHull.stl; visual mesh filename=package://klampt/meshes/7_7_scara_pince_doigt_optimized.stl
- added link pince_base, mass 0.1; collision mesh filename=package://klampt/meshes/7_7_scara_pince_base_convexHull.stl; visual mesh filename=package://klampt/meshes/7_7_scara_pince_base_optimized.stl
- added link poignet, mass 0.1; collision mesh filename=package://klampt/meshes/7_5_scara_poignet_convexHull.stl; visual mesh filename=package://klampt/meshes/7_5_scara_poignet_optimized.stl
- link electrique: geometry collision mesh filename=package://klampt/meshes/5_ZoneElec_only_convexHull.stl; visual mesh filename=package://klampt/meshes/5_ZoneElec_optimized.stl
- link stockage: geometry collision mesh filename=package://klampt/meshes/3_ZoneStockageV6_only_optimized.stl; visual mesh filename=package://klampt/meshes/3_ZoneStockageV6_optimized.stl
Joints:
- removed joint externe_poigner
- removed joint poigner_verin
- added joint externe_poignet: type revolute, parent externe, child poignet, origin xyz=0.29117 0.13275 0.030 rpy=0.0 0.0 0.0, axis 0.0 0.0 1.0, limit lower=-6 upper=6 effort=0.0 velocity=0.0
- added joint pince_doigt1: type revolute, parent pince_base, child doigt1, origin xyz=0.02405 0.07176 0.05466 rpy=0.0 2.094 0.0, axis 0.0 0.0 1.0, limit lower=0 upper=0.8346 effort=0.0 velocity=0.0
- added joint pince_doigt2: type revolute, parent pince_base, child doigt2, origin xyz=-0.05936 0.07176 -0.0065 rpy=0.0 0.0 0.0, axis 0.0 0.0 1.0, limit lower=0 upper=0.8346 effort=0.0 velocity=0.0, mimic joint=pince_doigt1 multiplier=1 offset=0
- added joint pince_doigt3: type revolute, parent pince_base, child doigt3, origin xyz=0.03531 0.07176 -0.04816 rpy=0.0 -2.094 0.0, axis 0.0 0.0 1.0, limit lower=0 upper=0.8346 effort=0.0 velocity=0.0, mimic joint=pince_doigt1 multiplier=1 offset=0
- added joint poignet_verin: type prismatic, parent poignet, child verin, origin xyz=0.0 0.0 -0.083 rpy=0.0 0.0 0.0, axis 0.0 0.0 1.0, limit lower=-0.15 upper=0.0 effort=0.0 velocity=0.0
- joint verin_pince: child pince -> pince_base

Commit message: klampt : verin_pince joint problem fixed

File: klampt/urdf/sysmap2_ros.urdf (robot description, URDF)
Before this commit: robot sysmap, 16 links, 15 joints
Joints:
- joint verin_pince: origin xyz=0.0 0.0 -0.025 rpy=-1.57 0.0 0.0 -> xyz=0.0 0.0 -0.025 rpy=-1.57 0.0 0.74

Commit message: klampt : add boite + couvercle cf Mathis Da

File: klampt/urdf/sysmap2_ros.urdf (robot description, URDF)
Before this commit: robot sysmap, 16 links, 15 joints
Links:
- removed link stockage
- added link stockage_boite; collision mesh filename=package://klampt/meshes/3_ZoneStockage_boite_convexHull.stl scale=0.001 0.001 0.001; visual mesh filename=package://klampt/meshes/3_ZoneStockage_boite_optimized.stl scale=0.001 0.001 0.001
- added link stockage_boite2; collision mesh filename=package://klampt/meshes/3_ZoneStockage_boite_convexHull.stl scale=0.001 0.001 0.001; visual mesh filename=package://klampt/meshes/3_ZoneStockage_boite_optimized.stl scale=0.001 0.001 0.001
- added link stockage_boite3; collision mesh filename=package://klampt/meshes/3_ZoneStockage_boite_convexHull.stl scale=0.001 0.001 0.001; visual mesh filename=package://klampt/meshes/3_ZoneStockage_boite_optimized.stl scale=0.001 0.001 0.001
- added link stockage_couvercle; collision mesh filename=package://klampt/meshes/3_ZoneStockage_couvercle_convexHull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 scale=0.001 0.001 0.001; visual mesh filename=package://klampt/meshes/3_ZoneStockage_couvercle_optimized.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 scale=0.001 0.001 0.001
- added link stockage_couvercle2; collision mesh filename=package://klampt/meshes/3_ZoneStockage_couvercle_convexHull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 scale=0.001 0.001 0.001; visual mesh filename=package://klampt/meshes/3_ZoneStockage_couvercle_optimized.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 scale=0.001 0.001 0.001
- added link stockage_couvercle3; collision mesh filename=package://klampt/meshes/3_ZoneStockage_couvercle_convexHull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 scale=0.001 0.001 0.001; visual mesh filename=package://klampt/meshes/3_ZoneStockage_couvercle_optimized.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 scale=0.001 0.001 0.001
- link interne: geometry collision mesh filename=package://klampt/meshes/7_3_scara_interne_convexHull.stl; visual mesh filename=package://klampt/meshes/7_3_scara_interne_optimized.stl
Joints:
- removed joint platine_stockage
- added joint platine_stockageBoite: type fixed, parent platine, child stockage_boite, origin xyz=-0.2789 -0.06397 0.0 rpy=1.57 0.0 -1.57
- added joint platine_stockageBoite2: type fixed, parent platine, child stockage_boite2, origin xyz=-0.2789 0.05803 0.0 rpy=1.57 0.0 -1.57
- added joint platine_stockageBoite3: type fixed, parent platine, child stockage_boite3, origin xyz=-0.2789 0.18003 0.0 rpy=1.57 0.0 -1.57
- added joint stockageBoite_couvercle: type revolute, parent stockage_boite, child stockage_couvercle, origin xyz=-0.0185 0.1203 0.1528 rpy=-0.117 0.0 0.0, axis -1.0 0.0 0.0, limit lower=0.0 upper=1.453 effort=0.0 velocity=0.0
- added joint stockageBoite_couvercle2: type revolute, parent stockage_boite2, child stockage_couvercle2, origin xyz=-0.0185 0.1203 0.1528 rpy=-0.117 0.0 0.0, axis -1.0 0.0 0.0, limit lower=0.0 upper=1.453 effort=0.0 velocity=0.0
- added joint stockageBoite_couvercle3: type revolute, parent stockage_boite3, child stockage_couvercle3, origin xyz=-0.0185 0.1203 0.1528 rpy=-0.117 0.0 0.0, axis -1.0 0.0 0.0, limit lower=0.0 upper=1.453 effort=0.0 velocity=0.0
- joint externe_poignet: limit lower=-6 upper=6 effort=0.0 velocity=0.0 -> lower=-3 upper=3 effort=0.0 velocity=0.0

Commit message: klampt : butés aproximatives done

File: klampt/urdf/sysmap2_ros.urdf (robot description, URDF)
Before this commit: robot sysmap, 21 links, 20 joints
Joints:
- joint base_colonne: limit lower=-6 upper=6 effort=0.0 velocity=0.0 -> lower=0 upper=6.35 effort=0.0 velocity=0.0; origin xyz=0.0 0.0 0.03 rpy=0.0 0.0 0.0 -> xyz=0.0 0.0 0.03 rpy=0.0 0.0 -5.4044
- joint externe_poignet: axis 0.0 0.0 1.0 -> 0.0 0.0 -1.0; limit lower=-3 upper=3 effort=0.0 velocity=0.0 -> lower=0 upper=6.35 effort=0.0 velocity=0.0; origin xyz=0.29117 0.13275 0.030 rpy=0.0 0.0 0.0 -> xyz=0.29117 0.13275 0.030 rpy=0.0 0.0 2.36
- joint interne_externe: axis 0.0 0.0 1.0 -> 0.0 0.0 -1.0; limit lower=-2.1 upper=2.56 effort=0.0 velocity=0.0 -> lower=0.0 upper=4.66 effort=0.0 velocity=0.0; origin xyz=0.214559 0.163904 -0.005 rpy=0.0 0.0 0.0 -> xyz=0.214559 0.163904 -0.005 rpy=0.0 0.0 2.56

Commit message: klampt : update URDF and meshes

File: klampt/urdf/sysmap2_ros.urdf (robot description, URDF)
Before this commit: robot sysmap, 21 links, 20 joints
Links:
- added link electrique_plateau; collision mesh filename=package://klampt/meshes/5_ZoneElec_plateau_optimized.stl; visual mesh filename=package://klampt/meshes/5_ZoneElec_plateau_optimized.stl
- link batterie: geometry collision mesh filename=package://klampt/meshes/6_ZoneBatterie.stl; visual mesh filename=package://klampt/meshes/6_ZoneBatterie.stl
- link electrique: geometry collision mesh filename=package://klampt/meshes/5_ZoneElec_convexHull.stl; visual mesh filename=package://klampt/meshes/5_ZoneElec_optimized.stl
Joints:
- added joint platine_electriquePlateau: type fixed, parent platine, child electrique_plateau, origin xyz=-0.1179 -0.004 0.0 rpy=0.0 0.0 0.0
- joint colonne_interne: limit lower=-0.2995 upper=0 effort=0.0 velocity=0.0 -> lower=-0.2789 upper=0 effort=0.0 velocity=0.0
- joint interne_externe: limit lower=0.0 upper=4.66 effort=0.0 velocity=0.0 -> lower=0.0 upper=4.54 effort=0.0 velocity=0.0; origin xyz=0.214559 0.163904 -0.005 rpy=0.0 0.0 2.56 -> xyz=0.214559 0.163904 -0.005 rpy=0.0 0.0 2.48
- joint poignet_verin: origin xyz=0.0 0.0 -0.083 rpy=0.0 0.0 0.0 -> xyz=0.0 0.0 -0.049 rpy=0.0 0.0 0.0

Commit message: klampt : redo collision of scara base

File: klampt/urdf/sysmap2_ros.urdf (robot description, URDF)
Before this commit: robot sysmap, 22 links, 21 joints
Links:
- link electrique_plateau: geometry collision mesh filename=package://klampt/meshes/5_ZoneElec_plateau_convexHull.stl; visual mesh filename=package://klampt/meshes/5_ZoneElec_plateau_optimized.stl

Commit message: klampt : base_colonne joint upper limit update

File: klampt/urdf/sysmap2_ros.urdf (robot description, URDF)
Before this commit: robot sysmap, 22 links, 21 joints
Joints:
- joint base_colonne: limit lower=0 upper=6.35 effort=0.0 velocity=0.0 -> lower=0 upper=6.13 effort=0.0 velocity=0.0

Commit message: moveit : change limit vitesse to 0.5rad and 0.1m

File: klampt/urdf/sysmap2_ros.urdf (robot description, URDF)
Before this commit: robot sysmap, 21 links, 20 joints
Links:
- added link aileron_camera; collision mesh filename=package://klampt/meshes/2_SupportAileron_camera_convexHull.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; visual mesh filename=package://klampt/meshes/2_SupportAileron_camera_optimized.s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
Joints:
- added joint platine_aileron_camera: type prismatic, parent platine, child aileron_camera, origin xyz=-0.42 0.042 -0.05 rpy=0.0 0.0 0.0, axis 0.0 0.0 1.0, limit lower=-0.05 upper=0.08 effort=0.0 velocity=0.0
- joint base_colonne: limit lower=0 upper=6.13 effort=0.0 velocity=0.0 -> lower=0 upper=6.13 effort=0.0 velocity=0.01
- joint colonne_interne: limit lower=-0.2789 upper=0 effort=0.0 velocity=0.0 -> lower=-0.2789 upper=0 effort=0.0 velocity=0.01
- joint externe_poignet: limit lower=0 upper=6.35 effort=0.0 velocity=0.0 -> lower=0 upper=6.35 effort=0.0 velocity=0.01
- joint interne_externe: limit lower=0.0 upper=4.54 effort=0.0 velocity=0.0 -> lower=0.0 upper=4.54 effort=0.0 velocity=0.01
- joint pince_doigt1: limit lower=0 upper=0.8346 effort=0.0 velocity=0.0 -> lower=0 upper=0.8346 effort=0.0 velocity=0.01
- joint pince_doigt2: limit lower=0 upper=0.8346 effort=0.0 velocity=0.0 -> lower=0 upper=0.8346 effort=0.0 velocity=0.01
- joint pince_doigt3: limit lower=0 upper=0.8346 effort=0.0 velocity=0.0 -> lower=0 upper=0.8346 effort=0.0 velocity=0.01
- joint poignet_verin: limit lower=-0.15 upper=0.0 effort=0.0 velocity=0.0 -> lower=-0.15 upper=0.0 effort=0.0 velocity=0.01

Commit message: global update
add moveit_liquide
add tempo to joystick pick drop and macro frottis
add all launch to moveit_hyperion/moveit_liquide demo2.launch
add all launch to vision all.launch
add rotation to vision
remove pince from vision pub and sub
set vision error tempo to 10s

File: klampt/urdf/sysmap2_ros.urdf (robot description, URDF)
Before this commit: robot sysmap, 22 links, 21 joints
Joints:
- joint base_colonne: limit lower=0 upper=6.13 effort=0.0 velocity=0.01 -> lower=0 upper=6.13 effort=0.0 velocity=0.6
- joint colonne_interne: limit lower=-0.2789 upper=0 effort=0.0 velocity=0.01 -> lower=-0.2789 upper=0 effort=0.0 velocity=0.05
- joint externe_poignet: limit lower=0 upper=6.35 effort=0.0 velocity=0.01 -> lower=0 upper=6.35 effort=0.0 velocity=0.6
- joint interne_externe: limit lower=0.0 upper=4.54 effort=0.0 velocity=0.01 -> lower=0.0 upper=4.54 effort=0.0 velocity=0.6
- joint pince_doigt1: limit lower=0 upper=0.8346 effort=0.0 velocity=0.01 -> lower=0 upper=0.8346 effort=0.0 velocity=0.6
- joint pince_doigt2: limit lower=0 upper=0.8346 effort=0.0 velocity=0.01 -> lower=0 upper=0.8346 effort=0.0 velocity=0.6
- joint pince_doigt3: limit lower=0 upper=0.8346 effort=0.0 velocity=0.01 -> lower=0 upper=0.8346 effort=0.0 velocity=0.6
- joint poignet_verin: limit lower=-0.15 upper=0.0 effort=0.0 velocity=0.01 -> lower=-0.15 upper=0.0 effort=0.0 velocity=0.15

File: klampt/urdf/sysmap_liquide.urdf (robot description, URDF)
Before this commit: robot sysmap, 18 links, 17 joints
Links:
- added link aileron_camera; collision mesh filename=package://klampt/meshes/2_SupportAileron_camera_convexHull.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; visual mesh filename=package://klampt/meshes/2_SupportAileron_camera_optimized.s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
Joints:
- added joint platine_aileron_camera: type prismatic, parent platine, child aileron_camera, origin xyz=-0.42 0.042 -0.05 rpy=0.0 0.0 0.0, axis 0.0 0.0 1.0, limit lower=-0.05 upper=0.08 effort=0.0 velocity=0.0
- joint base_colonne: limit lower=0 upper=6.13 effort=0.0 velocity=0.0 -> lower=0 upper=6.13 effort=0.0 velocity=0.6
- joint colonne_interne: limit lower=-0.2789 upper=0 effort=0.0 velocity=0.0 -> lower=-0.2789 upper=0 effort=0.0 velocity=0.05
- joint externe_poignet: limit lower=0 upper=6.35 effort=0.0 velocity=0.0 -> lower=0 upper=6.35 effort=0.0 velocity=0.6
- joint interne_externe: limit lower=0.0 upper=4.54 effort=0.0 velocity=0.0 -> lower=0.0 upper=4.54 effort=0.0 velocity=0.6
- joint pince_doigt1: limit lower=0 upper=0.8346 effort=0.0 velocity=0.0 -> lower=0 upper=0.8346 effort=0.0 velocity=0.6
- joint pince_doigt2: limit lower=0 upper=0.8346 effort=0.0 velocity=0.0 -> lower=0 upper=0.8346 effort=0.0 velocity=0.6
- joint pince_doigt3: limit lower=0 upper=0.8346 effort=0.0 velocity=0.0 -> lower=0 upper=0.8346 effort=0.0 velocity=0.6
- joint platine_stockageLiquide: axis (none) -> 0.0 0.0 1.0; limit (none) -> lower=0 upper=0.1 effort=0.0 velocity=0.01; type fixed -> prismatic
- joint platine_stockageLiquide2: axis (none) -> 0.0 0.0 1.0; limit (none) -> lower=0 upper=0.1 effort=0.0 velocity=0.01; type fixed -> prismatic
- joint platine_stockageLiquide3: axis (none) -> 0.0 0.0 1.0; limit (none) -> lower=0 upper=0.1 effort=0.0 velocity=0.01; type fixed -> prismatic
- joint poignet_verin: limit lower=-0.15 upper=0.0 effort=0.0 velocity=0.0 -> lower=-0.15 upper=0.0 effort=0.0 velocity=0.15

File: moveit_liquide/config/gazebo_sysmap.urdf (robot description, URDF)
Before this commit: robot sysmap, 22 links, 21 joints
Links:
- removed link stockage_boite
- removed link stockage_boite2
- removed link stockage_boite3
- removed link stockage_couvercle
- removed link stockage_couvercle2
- removed link stockage_couvercle3
- added link stockage_liquide, mass 0.1; collision mesh filename=package://klampt/meshes/3_ZoneStockage_liquide_convexHull.s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; visual mesh filename=package://klampt/meshes/3_ZoneStockage_liquide_optimized.stl
- added link stockage_liquide2, mass 0.1; collision mesh filename=package://klampt/meshes/3_ZoneStockage_liquide_convexHull.s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; visual mesh filename=package://klampt/meshes/3_ZoneStockage_liquide_optimized.stl
- added link stockage_liquide3, mass 0.1; collision mesh filename=package://klampt/meshes/3_ZoneStockage_liquide_convexHull.s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; visual mesh filename=package://klampt/meshes/3_ZoneStockage_liquide_optimized.stl
Joints:
- removed joint platine_stockageBoite
- removed joint platine_stockageBoite2
- removed joint platine_stockageBoite3
- removed joint stockageBoite_couvercle
- removed joint stockageBoite_couvercle2
- removed joint stockageBoite_couvercle3
- added joint platine_stockageLiquide: type prismatic, parent platine, child stockage_liquide, origin xyz=-0.2789 -0.06397 0.0 rpy=0.0 0.0 0.0, axis 0.0 0.0 1.0, limit lower=0 upper=0 effort=0.0 velocity=0.01
- added joint platine_stockageLiquide2: type prismatic, parent platine, child stockage_liquide2, origin xyz=-0.2789 0.05803 0.0 rpy=0.0 0.0 0.0, axis 0.0 0.0 1.0, limit lower=0 upper=0 effort=0.0 velocity=0.01
- added joint platine_stockageLiquide3: type prismatic, parent platine, child stockage_liquide3, origin xyz=-0.2789 0.18003 0.0 rpy=0.0 0.0 0.0, axis 0.0 0.0 1.0, limit lower=0 upper=0 effort=0.0 velocity=0.01

Commit message: change urdf name

File: klampt/urdf/sysmap2_ros.urdf (robot description, URDF)
Before this commit: robot sysmap, 22 links, 21 joints
Joints:
- removed joint base_colonne
- removed joint colonne_interne
- removed joint externe_poignet
- removed joint interne_externe
- removed joint pince_doigt1
- removed joint poignet_verin
- added joint base_rotation: type revolute, parent base, child colonne, origin xyz=0.0 0.0 0.03 rpy=0.0 0.0 -5.4044, axis 0.0 0.0 1.0, limit lower=0 upper=6.13 effort=0.0 velocity=0.6
- added joint epaule_rotation: type revolute, parent interne, child externe, origin xyz=0.214559 0.163904 -0.005 rpy=0.0 0.0 2.48, axis 0.0 0.0 -1.0, limit lower=0.0 upper=4.54 effort=0.0 velocity=0.6
- added joint epaule_translation: type prismatic, parent colonne, child interne, origin xyz=0.0 0.0 0.391 rpy=0.0 0.0 0.0, axis 0.0 0.0 1.0, limit lower=-0.2789 upper=0 effort=0.0 velocity=0.05
- added joint fermeture_pince_ouverture: type revolute, parent pince_base, child doigt1, origin xyz=0.02405 0.07176 0.05466 rpy=0.0 2.094 0.0, axis 0.0 0.0 1.0, limit lower=0 upper=0.8346 effort=0.0 velocity=0.6
- added joint pince_rotation: type revolute, parent externe, child poignet, origin xyz=0.29117 0.13275 0.030 rpy=0.0 0.0 2.36, axis 0.0 0.0 -1.0, limit lower=0 upper=5.45 effort=0.0 velocity=0.6
- added joint verin: type prismatic, parent poignet, child verin, origin xyz=0.0 0.0 -0.049 rpy=0.0 0.0 0.0, axis 0.0 0.0 1.0, limit lower=-0.15 upper=0.0 effort=0.0 velocity=0.15
- joint pince_doigt2: mimic joint=pince_doigt1 multiplier=1 offset=0 -> joint=fermeture_pince_ouverture multiplier=1 offset=0
- joint pince_doigt3: mimic joint=pince_doigt1 multiplier=1 offset=0 -> joint=fermeture_pince_ouverture multiplier=1 offset=0

File: moveit_hyperion/config/gazebo_sysmap.urdf (robot description, URDF)
Before this commit: robot sysmap, 22 links, 21 joints
Joints:
- removed joint base_colonne
- removed joint colonne_interne
- removed joint externe_poignet
- removed joint interne_externe
- removed joint pince_doigt1
- removed joint poignet_verin
- added joint base_rotation: type revolute, parent base, child colonne, origin xyz=0.0 0.0 0.03 rpy=0.0 0.0 -5.4044, axis 0.0 0.0 1.0, limit lower=0 upper=6.13 effort=0.0 velocity=0.6
- added joint epaule_rotation: type revolute, parent interne, child externe, origin xyz=0.214559 0.163904 -0.005 rpy=0.0 0.0 2.48, axis 0.0 0.0 -1.0, limit lower=0.0 upper=4.54 effort=0.0 velocity=0.6
- added joint epaule_translation: type prismatic, parent colonne, child interne, origin xyz=0.0 0.0 0.391 rpy=0.0 0.0 0.0, axis 0.0 0.0 1.0, limit lower=-0.2789 upper=0 effort=0.0 velocity=0.05
- added joint fermeture_pince_ouverture: type revolute, parent pince_base, child doigt1, origin xyz=0.02405 0.07176 0.05466 rpy=0.0 2.094 0.0, axis 0.0 0.0 1.0, limit lower=0 upper=0.8346 effort=0.0 velocity=0.6
- added joint pince_rotation: type revolute, parent externe, child poignet, origin xyz=0.29117 0.13275 0.030 rpy=0.0 0.0 2.36, axis 0.0 0.0 -1.0, limit lower=0 upper=5.45 effort=0.0 velocity=0.6
- added joint verin: type prismatic, parent poignet, child verin, origin xyz=0.0 0.0 -0.049 rpy=0.0 0.0 0.0, axis 0.0 0.0 1.0, limit lower=-0.15 upper=0.0 effort=0.0 velocity=0.15
- joint pince_doigt2: mimic joint=pince_doigt1 multiplier=1 offset=0 -> joint=fermeture_pince_ouverture multiplier=1 offset=0
- joint pince_doigt3: mimic joint=pince_doigt1 multiplier=1 offset=0 -> joint=fermeture_pince_ouverture multiplier=1 offset=0
